File: EXLROM/EXLROM_256Kbit/EXLROM_256kbit.kicad_sch (KiCad schematic)
At the start: 3 parts, among them J1 EXL100 Cartridge, U1 27C256

Commit message: Added ROMs & corrected silkscreen
Parts:
- C1: value 10nF -> 100nF
Changed lines of the file:
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@@
 			)
 		)
-		(property "Value" "10nF"
+		(property "Value" "100nF"
 			(at 127 76.1999 0)
 			(effects
