File: EXLROM/EXLROM_4Mbit/EXLROM_4Mbit.kicad_sch (KiCad schematic)
At the start: 8 parts, among them J1 EXL100 Cartridge, SW1 SW_DIP_x04, U1 27C040

Commit message: Added ROMs & corrected silkscreen
Parts:
- C1: value 10nF -> 100nF
Changed lines of the file:
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@@
 			)
 		)
-		(property "Value" "10nF"
+		(property "Value" "100nF"
 			(at 127 76.1999 0)
 			(effects
